File: schematic/Sheet01_Title.kicad_sch (KiCad schematic)
At the start: 0 parts

Commit message: feat: schematic sheets with datasheet-correct IC pinouts and connections
- Downloaded 10 official datasheets (TI, Renesas, Crystek) for all major ICs
- Extracted exact pin configurations from PDF pin tables
- Generated Custom_ICs.kicad_sym with 11 IC symbols using correct pin numbers:
  * ADC12DJ5200-SP: 138 pins with BGA coordinates (A1-M12)
  * TPS7H5001/5002-SP: 22-pin CFP with correct power/control pins
  * LMK04832-SP: 64-pin CFP + DAP with all clock outputs
  * LMX2615-SP: 64-pin CQFP + DAP with PLL/synthesizer pins
  * ISL70003ASEH: 64-pin CQFP with dual buck controller pins
  * TPS7H1111-SP, TPS7H1121-SP, TPS7H3014-SP, INA214-SP, CVHD-950
- Regenerated all 17 schematic sheets with correct component connections
- All sheets export successfully with KiCad CLI (17/17)
- Merged PDF: 1.3MB, 17 pages
Other:
- title: X-Band Digital Module 20x20cm -> X-Band Digital Module 20x20cm - Title
Changed lines of the file:
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@@
   (paper "A3")
   (title_block
-    (title "X-Band Digital Module 20x20cm")
+    (title "X-Band Digital Module 20x20cm - Title")
     (date "2026-09-10")
     (rev "1.0")
