File: schematic/Sheet05_Clock.kicad_sch (KiCad schematic)
At the start: 41 parts, among them U3 LMX2615-SP, U4 LMK04832-SP, Y1 CVHD-950-122.88MHz

Commit message: feat: connect ALL passive components and fix clock routing
- Added PASSIVE_TOPOLOGY dict mapping 139 passives to their nets
- Passive pin endpoints now get global_labels (was 0 connected, now 138)
- R38 intentionally GND-GND (RECAL_EN pull-down)
- Fixed LMK clock output mapping: CLKout0→ADC_CLK_P, CLKout2→FPGA_REFCLK_P, etc.
- Fixed TPS7H5001-SP SYNC pin collision with LMX_SYNC
- Total connections: 867 pins (up from 641)
- Cross-sheet nets: 52
- Power rails: VIN(33), +3V3(98), GND(228) all with decoupling
- JESD204C: U1↔U2 on 4 lanes ✓
- SPI: U1↔U2↔U3↔U4 ✓
- Clock: LMK→ADC (CLK+SYSREF), LMK→FPGA (REF+SPW) ✓
Parts:
- removed R30, R39: 1k, R_0402, symbol Device:R
- added R30 (x2): 1k, R_0402, symbol Device:R
Connections:
- net +3V3: now also C42.1, C43.1, C44.1, C45.1, C46.1, C47.1, C48.1, C49.1, C50.1, C51.1, C54.1, C55.1, C56.1, C57.1, C58.1, C59.1, C60.1, C61.1, C62.1, C63.1, C64.1, C65.1, C66.1, C67.1
- net GND: now also C40.2, C41.2, C42.2, C43.2, C44.2, C45.2, C46.2, C47.2, C48.2, C49.2, C50.2, C51.2, C52.2, C53.2, C54.2, C55.2, C56.2, C57.2, C58.2, C59.2, C60.2, C61.2, C62.2, C63.2, C64.2, C65.2, C66.2, C67.2, R31.2, R32.2, R33.2, R34.2, R35.2, R36.2, R37.2, R38.1, R38.2, R30.2, R30.2
- net PLL_CPOUT1: now also C52.1, C53.1
- net LMX_FS3: now reaches R33.1
- net LMX_FS1: now reaches R31.1
- net LMX_FS4: now reaches R34.1
- net LMX_FS6: now reaches R36.1
- net LMX_FS5: now reaches R35.1
- net +2V5_LDO: now reaches C41.1
- net +2V5_LDO: now also C40.1
- net LMX_FS7: now reaches R37.1
- net LMX_FS2: now reaches R32.1
- net LMK_CLK0_N renamed ADC_CLK_N
- net LMK_CLK0_P renamed ADC_CLK_P
- net LMK_CLK1_N renamed ADC_SYSREF_N
- net LMK_CLK1_P renamed ADC_SYSREF_P
- net LMK_CLK2_N renamed FPGA_REFCLK_N
- net LMK_CLK2_P renamed FPGA_REFCLK_P
- net LMK_CLK3_N renamed FPGA_SPWCLK_N
- net LMK_CLK3_P renamed FPGA_SPWCLK_P
- new net LMX_FS0: R30.1, R30.1
Changed lines of the file:
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@@
   )  (symbol (lib_id "Device:R") (at 140 120 0) (unit 1)
     (in_bom yes) (on_board yes)
-    (property "Reference" "R39" (at 140 110 0) (effects (font (size 1.27 1.27))))
+    (property "Reference" "R30" (at 140 110 0) (effects (font (size 1.27 1.27))))
     (property "Value" "1k" (at 140 130 0) (effects (font (size 1.27 1.27))))
     (property "Footprint" "R_0402" (at 140 120 0) (effects (font (size 1.27 1.27)) hide))
@@
   (global_label "CLKIN_SEL0" (at 379.6800 74.9200 0) (effects (font (size 1.27 1.27))))
   (global_label "CLKIN_SEL1" (at 379.6800 76.1900 0) (effects (font (size 1.27 1.27))))
-  (global_label "LMK_CLK0_P" (at 420.3200 58.4100 0) (effects (font (size 1.27 1.27))))
-  (global_label "LMK_CLK0_N" (at 420.3200 59.6800 0) (effects (font (size 1.27 1.27))))
-  (global_label "LMK_CLK1_P" (at 420.3200 60.9500 0) (effects (font (size 1.27 1.27))))
-  (global_label "LMK_CLK1_N" (at 420.3200 62.2200 0) (effects (font (size 1.27 1.27))))
-  (global_label "LMK_CLK2_P" (at 420.3200 63.4900 0) (effects (font (size 1.27 1.27))))
-  (global_label "LMK_CLK2_N" (at 420.3200 64.7600 0) (effects (font (size 1.27 1.27))))
-  (global_label "LMK_CLK3_P" (at 420.3200 66.0300 0) (effects (font (size 1.27 1.27))))
-  (global_label "LMK_CLK3_N" (at 420.3200 67.3000 0) (effects (font (size 1.27 1.27))))
+  (global_label "ADC_CLK_P" (at 420.3200 58.4100 0) (effects (font (size 1.27 1.27))))
+  (global_label "ADC_CLK_N" (at 420.3200 59.6800 0) (effects (font (size 1.27 1.27))))
+  (global_label "ADC_SYSREF_P" (at 420.3200 60.9500 0) (effects (font (size 1.27 1.27))))
+  (global_label "ADC_SYSREF_N" (at 420.3200 62.2200 0) (effects (font (size 1.27 1.27))))
+  (global_label "FPGA_REFCLK_P" (at 420.3200 63.4900 0) (effects (font (size 1.27 1.27))))
+  (global_label "FPGA_REFCLK_N" (at 420.3200 64.7600 0) (effects (font (size 1.27 1.27))))
+  (global_label "FPGA_SPWCLK_P" (at 420.3200 66.0300 0) (effects (font (size 1.27 1.27))))
+  (global_label "FPGA_SPWCLK_N" (at 420.3200 67.3000 0) (effects (font (size 1.27 1.27))))
   (global_label "LMK_CLK4_P" (at 420.3200 68.5700 0) (effects (font (size 1.27 1.27))))
   (global_label "LMK_CLK4_N" (at 420.3200 69.8400 0) (effects (font (size 1.27 1.27))))
@@
   (global_label "GND" (at 410.7950 106.6701 0) (effects (font (size 1.27 1.27))))
   (global_label "GND" (at 412.0650 106.6701 0) (effects (font (size 1.27 1.27))))
+  (global_label "+2V5_LDO" (at 60.0000 56.1900 0) (effects (font (size 1.27 1.27))))
+  (global_label "GND" (at 60.0000 63.8100 0) (effects (font (size 1.27 1.27))))
+  (global_label "+2V5_LDO" (at 60.0000 66.1900 0) (effects (font (size 1.27 1.27))))
+  (global_label "GND" (at 60.0000 73.8100 0) (effects (font (size 1.27 1.27))))
+  (global_label "+3V3" (at 140.0000 16.1900 0) (effects (font (size 1.27 1.27))))
+  (global_label "GND" (at 140.0000 23.8100 0) (effects (font (size 1.27 1.27))))
+  (global_label "+3V3" (at 170.0000 16.1900 0) (effects (font (size 1.27 1.27))))
+  (global_label "GND" (at 170.0000 23.8100 0) (effects (font (size 1.27 1.27))))
+  (global_label "+3V3" (at 200.0000 16.1900 0) (effects (font (size 1.27 1.27))))
+  (global_label "GND" (at 200.0000 23.8100 0) (effects (font (size 1.27 1.27))))
+  (global_label "+3V3" (at 230.0000 16.1900 0) (effects (font (size 1.27 1.27))))
+  (global_label "GND" (at 230.0000 23.8100 0) (effects (font (size 1.27 1.27))))
+  (global_label "+3V3" (at 260.0000 16.1900 0) (effects (font (size 1.27 1.27))))
+  (global_label "GND" (at 260.0000 23.8100 0) (effects (font (size 1.27 1.27))))
+  (global_label "+3V3" (at 140.0000 36.1900 0) (effects (font (size 1.27 1.27))))
+  (global_label "GND" (at 140.0000 43.8100 0) (effects (font (size 1.27 1.27))))
+  (global_label "+3V3" (at 170.0000 36.1900 0) (effects (font (size 1.27 1.27))))
+  (global_label "GND" (at 170.0000 43.8100 0) (effects (font (size 1.27 1.27))))
+  (global_label "+3V3" (at 200.0000 36.1900 0) (effects (font (size 1.27 1.27))))
+  (global_label "GND" (at 200.0000 43.8100 0) (effects (font (size 1.27 1.27))))
+  (global_label "+3V3" (at 230.0000 36.1900 0) (effects (font (size 1.27 1.27))))
+  (global_label "GND" (at 230.0000 43.8100 0) (effects (font (size 1.27 1.27))))
+  (global_label "+3V3" (at 260.0000 36.1900 0) (effects (font (size 1.27 1.27))))
+  (global_label "GND" (at 260.0000 43.8100 0) (effects (font (size 1.27 1.27))))
+  (global_label "PLL_CPOUT1" (at 280.0000 56.1900 0) (effects (font (size 1.27 1.27))))
+  (global_label "GND" (at 280.0000 63.8100 0) (effects (font (size 1.27 1.27))))
+  (global_label "PLL_CPOUT1" (at 280.0000 71.1900 0) (effects (font (size 1.27 1.27))))
+  (global_label "GND" (at 280.0000 78.8100 0) (effects (font (size 1.27 1.27))))
+  (global_label "LMX_FS0" (at 280.0000 86.1900 0) (effects (font (size 1.27 1.27))))
+  (global_label "GND" (at 280.0000 93.8100 0) (effects (font (size 1.27 1.27))))
+  (global_label "LMX_FS0" (at 140.0000 116.1900 0) (effects (font (size 1.27 1.27))))
+  (global_label "GND" (at 140.0000 123.8100 0) (effects (font (size 1.27 1.27))))
+  (global_label "LMX_FS1" (at 140.0000 126.1900 0) (effects (font (size 1.27 1.27))))
+  (global_label "GND" (at 140.0000 133.8100 0) (effects (font (size 1.27 1.27))))
+  (global_label "LMX_FS2" (at 140.0000 136.1900 0) (effects (font (size 1.27 1.27))))
+  (global_label "GND" (at 140.0000 143.8100 0) (effects (font (size 1.27 1.27))))
+  (global_label "LMX_FS3" (at 140.0000 146.1900 0) (effects (font (size 1.27 1.27))))
+  (global_label "GND" (at 140.0000 153.8100 0) (effects (font (size 1.27 1.27))))
+  (global_label "LMX_FS4" (at 140.0000 156.1900 0) (effects (font (size 1.27 1.27))))
+  (global_label "GND" (at 140.0000 163.8100 0) (effects (font (size 1.27 1.27))))
+  (global_label "LMX_FS5" (at 140.0000 166.1900 0) (effects (font (size 1.27 1.27))))
+  (global_label "GND" (at 140.0000 173.8100 0) (effects (font (size 1.27 1.27))))
+  (global_label "LMX_FS6" (at 140.0000 176.1900 0) (effects (font (size 1.27 1.27))))
+  (global_label "GND" (at 140.0000 183.8100 0) (effects (font (size 1.27 1.27))))
+  (global_label "LMX_FS7" (at 140.0000 186.1900 0) (effects (font (size 1.27 1.27))))
+  (global_label "GND" (at 140.0000 193.8100 0) (effects (font (size 1.27 1.27))))
+  (global_label "GND" (at 140.0000 196.1900 0) (effects (font (size 1.27 1.27))))
+  (global_label "GND" (at 140.0000 203.8100 0) (effects (font (size 1.27 1.27))))
+  (global_label "+3V3" (at 340.0000 6.1900 0) (effects (font (size 1.27 1.27))))
+  (global_label "GND" (at 340.0000 13.8100 0) (effects (font (size 1.27 1.27))))
+  (global_label "+3V3" (at 365.0000 6.1900 0) (effects (font (size 1.27 1.27))))
+  (global_label "GND" (at 365.0000 13.8100 0) (effects (font (size 1.27 1.27))))
+  (global_label "+3V3" (at 390.0000 6.1900 0) (effects (font (size 1.27 1.27))))
+  (global_label "GND" (at 390.0000 13.8100 0) (effects (font (size 1.27 1.27))))
+  (global_label "+3V3" (at 415.0000 6.1900 0) (effects (font (size 1.27 1.27))))
+  (global_label "GND" (at 415.0000 13.8100 0) (effects (font (size 1.27 1.27))))
+  (global_label "+3V3" (at 340.0000 21.1900 0) (effects (font (size 1.27 1.27))))
+  (global_label "GND" (at 340.0000 28.8100 0) (effects (font (size 1.27 1.27))))
+  (global_label "+3V3" (at 365.0000 21.1900 0) (effects (font (size 1.27 1.27))))
+  (global_label "GND" (at 365.0000 28.8100 0) (effects (font (size 1.27 1.27))))
+  (global_label "+3V3" (at 390.0000 21.1900 0) (effects (font (size 1.27 1.27))))
+  (global_label "GND" (at 390.0000 28.8100 0) (effects (font (size 1.27 1.27))))
+  (global_label "+3V3" (at 415.0000 21.1900 0) (effects (font (size 1.27 1.27))))
+  (global_label "GND" (at 415.0000 28.8100 0) (effects (font (size 1.27 1.27))))
+  (global_label "+3V3" (at 340.0000 36.1900 0) (effects (font (size 1.27 1.27))))
+  (global_label "GND" (at 340.0000 43.8100 0) (effects (font (size 1.27 1.27))))
+  (global_label "+3V3" (at 365.0000 36.1900 0) (effects (font (size 1.27 1.27))))
+  (global_label "GND" (at 365.0000 43.8100 0) (effects (font (size 1.27 1.27))))
+  (global_label "+3V3" (at 390.0000 36.1900 0) (effects (font (size 1.27 1.27))))
+  (global_label "GND" (at 390.0000 43.8100 0) (effects (font (size 1.27 1.27))))
+  (global_label "+3V3" (at 415.0000 36.1900 0) (effects (font (size 1.27 1.27))))
+  (global_label "GND" (at 415.0000 43.8100 0) (effects (font (size 1.27 1.27))))
+  (global_label "+3V3" (at 450.0000 6.1900 0) (effects (font (size 1.27 1.27))))
+  (global_label "GND" (at 450.0000 13.8100 0) (effects (font (size 1.27 1.27))))
+  (global_label "+3V3" (at 450.0000 21.1900 0) (effects (font (size 1.27 1.27))))
+  (global_label "GND" (at 450.0000 28.8100 0) (effects (font (size 1.27 1.27))))
   (sheet_instances (path "/" (page "1")))
 )
