File: schematic/Sheet12_LDO_2V5.kicad_sch (KiCad schematic)
At the start: 10 parts, among them U10 TPS7H1121-SP

Commit message: feat: connect ALL passive components and fix clock routing
- Added PASSIVE_TOPOLOGY dict mapping 139 passives to their nets
- Passive pin endpoints now get global_labels (was 0 connected, now 138)
- R38 intentionally GND-GND (RECAL_EN pull-down)
- Fixed LMK clock output mapping: CLKout0→ADC_CLK_P, CLKout2→FPGA_REFCLK_P, etc.
- Fixed TPS7H5001-SP SYNC pin collision with LMX_SYNC
- Total connections: 867 pins (up from 641)
- Cross-sheet nets: 52
- Power rails: VIN(33), +3V3(98), GND(228) all with decoupling
- JESD204C: U1↔U2 on 4 lanes ✓
- SPI: U1↔U2↔U3↔U4 ✓
- Clock: LMK→ADC (CLK+SYSREF), LMK→FPGA (REF+SPW) ✓
Connections:
- net +3V3: now also C110.1, C111.1, C112.1
- net GND: now also C110.2, C111.2, C112.2, C113.2, C114.2, C115.2, C116.2, R65.2
- net U10_FB: now also R64.2, R65.1
- net +2V5_LDO: now reaches R64.1
- net +2V5_LDO: now also C113.1, C114.1, C115.1
- net U10_STAB: now reaches C116.1
Changed lines of the file:
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@@
   (global_label "GND" (at 202.5400 93.9700 0) (effects (font (size 1.27 1.27))))
   (global_label "TPS7H1121-SP_VLDO" (at 203.8100 93.9700 0) (effects (font (size 1.27 1.27))))
+  (global_label "+3V3" (at 120.0000 36.1900 0) (effects (font (size 1.27 1.27))))
+  (global_label "GND" (at 120.0000 43.8100 0) (effects (font (size 1.27 1.27))))
+  (global_label "+3V3" (at 120.0000 51.1900 0) (effects (font (size 1.27 1.27))))
+  (global_label "GND" (at 120.0000 58.8100 0) (effects (font (size 1.27 1.27))))
+  (global_label "+3V3" (at 120.0000 66.1900 0) (effects (font (size 1.27 1.27))))
+  (global_label "GND" (at 120.0000 73.8100 0) (effects (font (size 1.27 1.27))))
+  (global_label "+2V5_LDO" (at 300.0000 36.1900 0) (effects (font (size 1.27 1.27))))
+  (global_label "GND" (at 300.0000 43.8100 0) (effects (font (size 1.27 1.27))))
+  (global_label "+2V5_LDO" (at 300.0000 51.1900 0) (effects (font (size 1.27 1.27))))
+  (global_label "GND" (at 300.0000 58.8100 0) (effects (font (size 1.27 1.27))))
+  (global_label "+2V5_LDO" (at 300.0000 66.1900 0) (effects (font (size 1.27 1.27))))
+  (global_label "GND" (at 300.0000 73.8100 0) (effects (font (size 1.27 1.27))))
+  (global_label "U10_STAB" (at 200.0000 116.1900 0) (effects (font (size 1.27 1.27))))
+  (global_label "GND" (at 200.0000 123.8100 0) (effects (font (size 1.27 1.27))))
+  (global_label "+2V5_LDO" (at 300.0000 86.1900 0) (effects (font (size 1.27 1.27))))
+  (global_label "U10_FB" (at 300.0000 93.8100 0) (effects (font (size 1.27 1.27))))
+  (global_label "U10_FB" (at 300.0000 106.1900 0) (effects (font (size 1.27 1.27))))
+  (global_label "GND" (at 300.0000 113.8100 0) (effects (font (size 1.27 1.27))))
   (sheet_instances (path "/" (page "1")))
 )
